Commit message: Delete notes for urdf files

File: sim_arm_panda_gazebo/PandaRobot/panda_ros2_gazebo/urdf/panda.urdf.xacro (robot description, xacro)
@@ -1,60 +1,10 @@
 <?xml version="1.0"?>
-<!--
-# ===================================== COPYRIGHT ===================================== #
-#                                                                                       #
-#  IFRA (Intelligent Flexible Robotics and Assembly) Group, CRANFIELD UNIVERSITY        #
-#  Created on behalf of the IFRA Group at Cranfield University, United Kingdom          #
-#  E-mail: IFRA@cranfield.ac.uk                                                         #
-#                                                                                       #
-#  Licensed under the Apache-2.0 License.                                               #
-#  You may not use this file except in compliance with the License.                     #
-#  You may obtain a copy of the License at: http://www.apache.org/licenses/LICENSE-2.0  #
-#                                                                                       #
-#  Unless required by applicable law or agreed to in writing, software distributed      #
-#  under the License is distributed on an "as-is" basis, without warranties or          #
-#  conditions of any kind, either express or implied. See the License for the specific  #
-#  language governing permissions and limitations under the License.                    #
-#                                                                                       #
-#  IFRA Group - Cranfield University                                                    #
-#  AUTHORS: Mikel Bueno Viso - Mikel.Bueno-Viso@cranfield.ac.uk                         #
-#           Seemal Asif      - s.asif@cranfield.ac.uk                                   #
-#           Phil Webb        - p.f.webb@cranfield.ac.uk                                 #
-#                                                                                       #
-#  Date: July, 2022.                                                                    #
-#                                                                                       #
-# ===================================== COPYRIGHT ===================================== #
-# ===================================== COPYRIGHT ===================================== #
-#                                                                                       #
-#  Some of the information used to build the ROS2 Panda-Robot .urdf files in this ROS2  #
-#  repository has been taken from the following resources:                              #
-#     - frankaemika/franka_ros2 -> https://github.com/frankaemika/franka_ros2.          #
-#       The original files can be found in the franka_description ROS2 package inside   #
-#       he franka_ros2 GitHub repository.                                               #
-#                                                                                       #
-#  AUTHOR: Franka Emika GmbH - support@franka.de                                        #
-#                                                                                       #
-#  Copyright 2021 Franka Emika GmbH                                                     #
-#  (ORIGINAL LICENSE) -> Licensed under the Apache-2.0 License.                         #
-#                                                                                       #
-#  CHANGES MADE:                                                                        #
-#  Robot information/specifications have been taken, and the code has been modified and #
-#  re-organised in accordance with the ros2_RobotSimulation standards.                  #
-#                                                                                       #
-# ===================================== COPYRIGHT ===================================== #
-# ======= CITE OUR WORK ======= #
-# You can cite our work with the following statement:
-# IFRA (2022) ROS2.0 ROBOT SIMULATION. URL: https://github.com/IFRA-Cranfield/ros2_RobotSimulation.
--->
 <robot xmlns:xacro="http://wiki.ros.org/xacro" name="panda">
-  <!-- ===== ARGUMENTS ===== -->
-  <!-- CELL LAYOUT:  -->
   <xacro:arg name="cell_layout_1" default="false"/>
   <xacro:property name="cell_layout_1" value="$(arg cell_layout_1)"/>
   <xacro:arg name="cell_layout_2" default="false"/>
   <xacro:property name="cell_layout_2" value="$(arg cell_layout_2)"/>
-  <!-- END-EFFECTOR:  -->
   <xacro:arg name="EE_no" default="false"/>
   <xacro:property name="EE_no" value="$(arg EE_no)"/>
-  <!-- Include XACRO-MACRO file of the PANDA ROBOT: -->
   <xacro:include filename="$(find panda_ros2_gazebo)/urdf/panda_macro.urdf.xacro"/>
   <xacro:panda
@@ -62,9 +12,5 @@
     EE_no="${EE_no}"
   />
-  <!-- Gazebo world link: -->
   <link name="world"/>
-  <!-- ========== ========== ========== ========== ========== ========== -->
-  <!-- CELL LAYOUT SELECTION: -->
-  <!-- CELL LAYOUT N1) PANDA ROBOT alone: -->
   <xacro:if value="${cell_layout_1}">
     <joint name="world-base_link-fixed" type="fixed">
@@ -73,5 +19,4 @@
     </joint>
   </xacro:if>
-  <!-- CELL LAYOUT N2) PANDA ROBOT on top of a pedestal: -->
   <xacro:if value="${cell_layout_2}">
     <link name='panda_base'>

File: sim_arm_panda_gazebo/PandaRobot/panda_ros2_gazebo/urdf/panda_macro.urdf.xacro (robot description, xacro)
@@ -1,58 +1,9 @@
 <?xml version="1.0"?>
-<!--
-# ===================================== COPYRIGHT ===================================== #
-#                                                                                       #
-#  IFRA (Intelligent Flexible Robotics and Assembly) Group, CRANFIELD UNIVERSITY        #
-#  Created on behalf of the IFRA Group at Cranfield University, United Kingdom          #
-#  E-mail: IFRA@cranfield.ac.uk                                                         #
-#                                                                                       #
-#  Licensed under the Apache-2.0 License.                                               #
-#  You may not use this file except in compliance with the License.                     #
-#  You may obtain a copy of the License at: http://www.apache.org/licenses/LICENSE-2.0  #
-#                                                                                       #
-#  Unless required by applicable law or agreed to in writing, software distributed      #
-#  under the License is distributed on an "as-is" basis, without warranties or          #
-#  conditions of any kind, either express or implied. See the License for the specific  #
-#  language governing permissions and limitations under the License.                    #
-#                                                                                       #
-#  IFRA Group - Cranfield University                                                    #
-#  AUTHORS: Mikel Bueno Viso - Mikel.Bueno-Viso@cranfield.ac.uk                         #
-#           Seemal Asif      - s.asif@cranfield.ac.uk                                   #
-#           Phil Webb        - p.f.webb@cranfield.ac.uk                                 #
-#                                                                                       #
-#  Date: July, 2022.                                                                    #
-#                                                                                       #
-# ===================================== COPYRIGHT ===================================== #
-# ===================================== COPYRIGHT ===================================== #
-#                                                                                       #
-#  Some of the information used to build the ROS2 Panda-Robot .urdf files in this ROS2  #
-#  repository has been taken from the following resources:                              #
-#     - frankaemika/franka_ros2 -> https://github.com/frankaemika/franka_ros2.          #
-#       The original files can be found in the franka_description ROS2 package inside   #
-#       he franka_ros2 GitHub repository.                                               #
-#                                                                                       #
-#  AUTHOR: Franka Emika GmbH - support@franka.de                                        #
-#                                                                                       #
-#  Copyright 2021 Franka Emika GmbH                                                     #
-#  (ORIGINAL LICENSE) -> Licensed under the Apache-2.0 License.                         #
-#                                                                                       #
-#  CHANGES MADE:                                                                        #
-#  Robot information/specifications have been taken, and the code has been modified and #
-#  re-organised in accordance with the ros2_RobotSimulation standards.                  #
-#                                                                                       #
-# ===================================== COPYRIGHT ===================================== #
-# ======= CITE OUR WORK ======= #
-# You can cite our work with the following statement:
-# IFRA (2022) ROS2.0 ROBOT SIMULATION. URL: https://github.com/IFRA-Cranfield/ros2_RobotSimulation.
--->
 <robot xmlns:xacro="http://wiki.ros.org/xacro">
-  <!-- XACRO-MACRO of PANDA ROBOT: -->
   <xacro:macro name="panda" params="prefix EE_no">
-    <!-- Load PANDA ROBOT TRANSMISSION file: -->
     <xacro:include filename="$(find panda_ros2_gazebo)/urdf/panda_transmission.xacro" />
     <xacro:panda_transmission
       prefix=""
     />
-    <!-- Load PANDA ROBOT ROS2_CONTROL file: -->
     <xacro:include filename="$(find panda_ros2_gazebo)/urdf/panda_ros2control.xacro" />
     <xacro:panda_ros2control initial_positions_file="$(find panda_ros2_gazebo)/urdf/initial_positions.yaml" EE_no="${EE_no}"
@@ -62,6 +13,4 @@
       prefix="camera"
     />
-    <!-- ***** PANDA ROBOT .urdf SERIAL CHAIN ***** -->
-    <!-- panda_link0 -->
     <link name="panda_link0">
       <inertial>
@@ -86,5 +35,4 @@
       </collision>
     </link>
-    <!-- panda_link1 -->
     <link name="panda_link1">
       <inertial>
@@ -109,5 +57,4 @@
       </collision>
     </link>
-    <!-- panda_joint1 -->
     <joint name="panda_joint1" type="revolute">
       <origin rpy="0 0 0" xyz="0 0 0.333"/>
@@ -118,5 +65,4 @@
       <dynamics damping="50.0" friction="1.0"/>
     </joint>
-    <!-- panda_link2 -->
     <link name="panda_link2">
       <inertial>
@@ -141,5 +87,4 @@
       </collision>
     </link>
-    <!-- panda_joint2 -->
     <joint name="panda_joint2" type="revolute">
       <origin rpy="-1.57079632679 0 0" xyz="0 0 0"/>
@@ -150,5 +95,4 @@
       <dynamics damping="50.0" friction="1.0"/>
     </joint>
-    <!-- panda_link3 -->
     <link name="panda_link3">
       <inertial>
@@ -173,5 +117,4 @@
       </collision>
     </link>
-    <!-- panda_joint3 -->
     <joint name="panda_joint3" type="revolute">
       <origin rpy="1.57079632679 0 0" xyz="0 -0.316 0"/>
@@ -182,5 +125,4 @@
       <dynamics damping="10.0" friction="1.0"/>
     </joint>
-    <!-- panda_link4-->
     <link name="panda_link4">
       <inertial>
@@ -205,5 +147,4 @@
       </collision>
     </link>
-    <!-- panda_joint4 -->
     <joint name="panda_joint4" type="revolute">
       <origin rpy="1.57079632679 0 0" xyz="0.0825 0 0"/>
@@ -212,8 +153,6 @@
       <axis xyz="0 0 1"/>
       <limit effort="87" lower="-3.0718" upper="0.0698" velocity="2.1750"/>
-      <!-- upper should be -0.0698, but that brakes simulation when initial position for this joint is 0.0 -->
       <dynamics damping="10.0" friction="1.0"/>
     </joint>
-    <!-- panda_link5 -->
     <link name="panda_link5">
       <inertial>
@@ -238,5 +177,4 @@
       </collision>
     </link>
-    <!-- panda_joint5 -->
     <joint name="panda_joint5" type="revolute">
       <origin rpy="-1.57079632679 0 0" xyz="-0.0825 0.384 0"/>
@@ -247,5 +185,4 @@
       <dynamics damping="5.0" friction="1.0"/>
     </joint>
-    <!-- panda_link6 -->
     <link name="panda_link6">
       <inertial>
@@ -270,7 +207,6 @@
       </collision>
     </link>
-    <!-- panda_joint6 -->
     <joint name="panda_joint6" type="revolute">
-      <origin rpy="1.57079632679 -1.57079632679 0" xyz="0 0 0"/> <!-- rpy="1.57079632679 0 0" -->
+      <origin rpy="1.57079632679 -1.57079632679 0" xyz="0 0 0"/>
       <parent link="panda_link5"/>
       <child link="panda_link6"/>
@@ -279,5 +215,4 @@
       <dynamics damping="5.0" friction="1.0"/>
     </joint>
-    <!-- panda_link7 -->
     <link name="panda_link7">
       <inertial>
@@ -302,7 +237,6 @@
       </collision>
     </link>
-    <!-- panda_joint7 -->
     <joint name="panda_joint7" type="revolute">
-      <origin rpy="1.57079632679 -0.7854 0" xyz="0.088 0 0"/> <!-- rpy="1.57079632679 0 0" -->
+      <origin rpy="1.57079632679 -0.7854 0" xyz="0.088 0 0"/>
       <parent link="panda_link6"/>
       <child link="panda_link7"/>
@@ -311,7 +245,5 @@
       <dynamics damping="1.0" friction="1.0"/>
     </joint>
-    <!-- panda_link8 -->
     <link name="panda_link8"/>
-    <!-- panda_joint8 -->
     <joint name="panda_joint8" type="fixed">
       <origin rpy="0 0 0" xyz="0 0 0.107"/>
@@ -320,5 +252,4 @@
       <axis xyz="0 0 0"/>
     </joint>
-    <!-- panda_hand -->
     <joint name="panda_hand_joint" type="fixed">
       <parent link="panda_link8"/>
@@ -348,5 +279,4 @@
       </collision>
     </link>
-  <!--camera_link-->
     <link name="camera_link">
       <collision>
@@ -371,7 +301,5 @@
       </inertial>
     </link>
-    <!--camera_joint-->
     <joint name="camera_joint" type="fixed">
-      <!-- <axis xyz="0 0 0" /> -->
       <origin xyz="0.02 -0.02 0.15" rpy="1.57079632679 -1.57079632679 0.785398163397"/>
       <parent link="panda_link7"/>
@@ -381,5 +309,4 @@
       <dynamics damping="1.0" friction="1.0"/>
     </joint>
-    <!-- panda_leftfinger -->
     <link name="panda_leftfinger">
       <inertial>
@@ -404,5 +331,4 @@
       </collision>
     </link>
-    <!-- panda_rightfinger -->
     <link name="panda_rightfinger">
       <inertial>
@@ -443,8 +369,6 @@
       <dynamics damping="1.0" friction="1.0"/>
     </joint>
-    <!-- End-Effector frame -->
     <link name="end_effector_frame">
       <inertial>
-        <!-- Dummy inertial parameters to avoid link lumping-->
         <mass value="0.01"/>
         <inertia ixx="0.0001" ixy="0.0" ixz="0.0" iyy="0.0001" iyz="0.0" izz="0.0001"/>

File: sim_arm_panda_gazebo/PandaRobot/panda_ros2_gazebo/urdf/panda_ros2control.xacro (robot description, xacro)
@@ -1,57 +1,8 @@
 <?xml version="1.0"?>
-<!--
-# ===================================== COPYRIGHT ===================================== #
-#                                                                                       #
-#  IFRA (Intelligent Flexible Robotics and Assembly) Group, CRANFIELD UNIVERSITY        #
-#  Created on behalf of the IFRA Group at Cranfield University, United Kingdom          #
-#  E-mail: IFRA@cranfield.ac.uk                                                         #
-#                                                                                       #
-#  Licensed under the Apache-2.0 License.                                               #
-#  You may not use this file except in compliance with the License.                     #
-#  You may obtain a copy of the License at: http://www.apache.org/licenses/LICENSE-2.0  #
-#                                                                                       #
-#  Unless required by applicable law or agreed to in writing, software distributed      #
-#  under the License is distributed on an "as-is" basis, without warranties or          #
-#  conditions of any kind, either express or implied. See the License for the specific  #
-#  language governing permissions and limitations under the License.                    #
-#                                                                                       #
-#  IFRA Group - Cranfield University                                                    #
-#  AUTHORS: Mikel Bueno Viso - Mikel.Bueno-Viso@cranfield.ac.uk                         #
-#           Seemal Asif      - s.asif@cranfield.ac.uk                                   #
-#           Phil Webb        - p.f.webb@cranfield.ac.uk                                 #
-#                                                                                       #
-#  Date: July, 2022.                                                                    #
-#                                                                                       #
-# ===================================== COPYRIGHT ===================================== #
-# ===================================== COPYRIGHT ===================================== #
-#                                                                                       #
-#  Some of the information used to build the ROS2 Panda-Robot .urdf files in this ROS2  #
-#  repository has been taken from the following resources:                              #
-#     - frankaemika/franka_ros2 -> https://github.com/frankaemika/franka_ros2.          #
-#       The original files can be found in the franka_description ROS2 package inside   #
-#       he franka_ros2 GitHub repository.                                               #
-#                                                                                       #
-#  AUTHOR: Franka Emika GmbH - support@franka.de                                        #
-#                                                                                       #
-#  Copyright 2021 Franka Emika GmbH                                                     #
-#  (ORIGINAL LICENSE) -> Licensed under the Apache-2.0 License.                         #
-#                                                                                       #
-#  CHANGES MADE:                                                                        #
-#  Robot information/specifications have been taken, and the code has been modified and #
-#  re-organised in accordance with the ros2_RobotSimulation standards.                  #
-#                                                                                       #
-# ===================================== COPYRIGHT ===================================== #
-# ======= CITE OUR WORK ======= #
-# You can cite our work with the following statement:
-# IFRA (2022) ROS2.0 ROBOT SIMULATION. URL: https://github.com/IFRA-Cranfield/ros2_RobotSimulation.
--->
 <robot xmlns:xacro="http://www.ros.org/wiki/xacro">
   <xacro:macro name="panda_ros2control" params="initial_positions_file EE_no" >
     <xacro:arg name="initial_positions_file" default="initial_positions.yaml" />
     <xacro:property name="initial_positions" value="${xacro.load_yaml(initial_positions_file)['initial_positions']}"/>
-    <!-- ROS2_CONTROL tag name: -->
     <xacro:property name="name" value="GazeboSystem"/>
-    <!-- ===== Gazebo ROS2_CONTROL plugin ===== -->
-    <!-- No End-Effector: -->
     <xacro:if value="${EE_no}">
       <gazebo>
@@ -62,12 +13,9 @@
       </gazebo>
     </xacro:if>
-    <!-- ========== ROS2 CONTROL ========== -->
     <ros2_control name="${name}" type="system">
       <hardware>
         <plugin>gazebo_ros2_control/GazeboSystem</plugin>
       </hardware>
-      <!-- panda_joint1 -->
       <joint name="panda_joint1">
-        <!-- <param name="initial_position">0.0</param> -->
         <command_interface name="position">
           <param name="min">-2.8973</param>
@@ -84,14 +32,12 @@
         <state_interface name="effort"/>
       </joint>
-      <!-- panda_joint2 -->
       <joint name="panda_joint2">
         <param name="initial_position">-0.785</param>
         <command_interface name="position">
-          <!-- <param name="min">-1.7628</param>
           <param name="max">1.7628</param>
         </command_interface>
         <command_interface name="velocity">
           <param name="min">-2.1750</param>
-          <param name="max">2.1750</param> -->
+          <param name="max">2.1750</param>
         </command_interface>
         <state_interface name="position">
@@ -101,7 +47,5 @@
         <state_interface name="effort"/>
       </joint>
-      <!-- panda_joint3 -->
       <joint name="panda_joint3">
-        <!-- <param name="initial_position">0.0</param> -->
         <command_interface name="position">
           <param name="min">-2.8973</param>
@@ -118,7 +62,5 @@
         <state_interface name="effort"/>
       </joint>
-      <!-- panda_joint4 -->
       <joint name="panda_joint4">
-        <!-- <param name="initial_position">-2.356</param> -->
         <command_interface name="position">
           <param name="min">-3.0718</param>
@@ -135,7 +77,5 @@
         <state_interface name="effort"/>
       </joint>
-      <!-- panda_joint5 -->
       <joint name="panda_joint5">
-        <!-- <param name="initial_position">0.0</param> -->
         <command_interface name="position">
           <param name="min">-2.8973</param>
@@ -152,10 +92,8 @@
         <state_interface name="effort"/>
       </joint>
-      <!-- panda_joint6 -->
       <joint name="panda_joint6">
-        <!-- <param name="initial_position">1.5708</param> -->
         <command_interface name="position">
-          <param name="min">-0.0175</param> <!-- ** -1.5883 -->
-          <param name="max">3.7525</param> <!-- ** 2.1817 -->
+          <param name="min">-0.0175</param>
+          <param name="max">3.7525</param>
         </command_interface>
         <command_interface name="velocity">
@@ -169,10 +107,8 @@
         <state_interface name="effort"/>
       </joint>
-      <!-- panda_joint7 -->
       <joint name="panda_joint7">
-        <!-- <param name="initial_position">0.785</param> -->
         <command_interface name="position">
-          <param name="min">-3.15</param> <!-- ** -3.935 -->
-          <param name="max">3.15</param> <!-- ** 2.365 -->
+          <param name="min">-3.15</param>
+          <param name="max">3.15</param>
         </command_interface>
         <command_interface name="velocity">
@@ -186,5 +122,4 @@
         <state_interface name="effort"/>
       </joint>
-      <!-- panda_finger_joint1 -->
       <joint name="panda_finger_joint1">
         <command_interface name="position">
@@ -200,5 +135,4 @@
         <state_interface name="effort"/>
       </joint>
-      <!-- panda_finger_joint2 -->
       <joint name="panda_finger_joint2">
         <command_interface name="position">
@@ -253,5 +187,4 @@
     <gazebo reference="end_effector_frame_fixed_joint">
       <preserveFixedJoint>true</preserveFixedJoint>
-      <!-- For compatibility with SDFormat < 4.4 -->
       <disableFixedJointLumping>true</disableFixedJointLumping>
     </gazebo>
